Commit message: common Gazebo xacro for waffle and burger

File: urdf/turtlebot3_burger.urdf.xacro (robot description, xacro)
@@ -1,13 +1,16 @@
 <?xml version="1.0" ?>
 <robot name="turtlebot3_burger" xmlns:xacro="http://ros.org/wiki/xacro">
+ <!-- Properties of burger -->
+ <xacro:property name="wheel_separation" value="0.160" />
+ <xacro:arg name="use_cam" default="false"/>
   <xacro:include filename="$(find turtlebot3_description)/urdf/common_properties.xacro"/>
-  <xacro:include filename="$(find turtlebot3_description)/urdf/turtlebot3_burger.gazebo.xacro"/>
-  <link name="base_footprint"/>
+  <xacro:include filename="$(find turtlebot3_description)/urdf/turtlebot3_gazebo.xacro"/>
+  <link name="$(arg prefix)base_footprint"/>
   <joint name="base_joint" type="fixed">
-    <parent link="base_footprint"/>
-    <child link="base_link"/>
+    <parent link="$(arg prefix)base_footprint"/>
+    <child link="$(arg prefix)base_link"/>
     <origin xyz="0.0 0.0 0.010" rpy="0 0 0"/>
   </joint>
-  <link name="base_link">
+  <link name="$(arg prefix)base_link">
     <visual>
       <origin xyz="-0.032 0 0.0" rpy="0 0 0"/>
@@ -32,10 +35,10 @@
   </link>
   <joint name="wheel_left_joint" type="continuous">
-    <parent link="base_link"/>
-    <child link="wheel_left_link"/>
+    <parent link="$(arg prefix)base_link"/>
+    <child link="$(arg prefix)wheel_left_link"/>
     <origin xyz="0.0 0.08 0.023" rpy="-1.57 0 0"/>
     <axis xyz="0 0 1"/>
   </joint>
-  <link name="wheel_left_link">
+  <link name="$(arg prefix)wheel_left_link">
     <visual>
       <origin xyz="0 0 0" rpy="1.57 0 0"/>
@@ -60,10 +63,10 @@
   </link>
   <joint name="wheel_right_joint" type="continuous">
-    <parent link="base_link"/>
-    <child link="wheel_right_link"/>
+    <parent link="$(arg prefix)base_link"/>
+    <child link="$(arg prefix)wheel_right_link"/>
     <origin xyz="0.0 -0.080 0.023" rpy="-1.57 0 0"/>
     <axis xyz="0 0 1"/>
   </joint>
-  <link name="wheel_right_link">
+  <link name="$(arg prefix)wheel_right_link">
     <visual>
       <origin xyz="0 0 0" rpy="1.57 0 0"/>
@@ -88,9 +91,9 @@
   </link>
   <joint name="caster_back_joint" type="fixed">
-    <parent link="base_link"/>
-    <child link="caster_back_link"/>
+    <parent link="$(arg prefix)base_link"/>
+    <child link="$(arg prefix)caster_back_link"/>
     <origin xyz="-0.081 0 -0.004" rpy="-1.57 0 0"/>
   </joint>
-  <link name="caster_back_link">
+  <link name="$(arg prefix)caster_back_link">
     <collision>
       <origin xyz="0 0.001 0" rpy="0 0 0"/>
@@ -108,15 +111,15 @@
   </link>
   <joint name="imu_joint" type="fixed">
-    <parent link="base_link"/>
-    <child link="imu_link"/>
+    <parent link="$(arg prefix)base_link"/>
+    <child link="$(arg prefix)imu_link"/>
     <origin xyz="-0.032 0 0.068" rpy="0 0 0"/>
   </joint>
-  <link name="imu_link"/>
+  <link name="$(arg prefix)imu_link"/>
   <joint name="scan_joint" type="fixed">
-    <parent link="base_link"/>
-    <child link="base_scan"/>
+    <parent link="$(arg prefix)base_link"/>
+    <child link="$(arg prefix)base_scan"/>
     <origin xyz="-0.032 0 0.172" rpy="0 0 0"/>
   </joint>
-  <link name="base_scan">
+  <link name="$(arg prefix)base_scan">
     <visual>
       <origin xyz="0 0 0.0" rpy="0 0 0"/>

File: urdf/turtlebot3_waffle.urdf.xacro (robot description, xacro)
@@ -1,6 +1,9 @@
 <?xml version="1.0" ?>
 <robot name="turtlebot3_waffle" xmlns:xacro="http://ros.org/wiki/xacro">
+ <!-- Properties of waffle -->
+ <xacro:property name="wheel_separation" value="0.287" />
+ <xacro:arg name="use_cam" default="false"/>
   <xacro:include filename="$(find turtlebot3_description)/urdf/common_properties.xacro"/>
-  <xacro:include filename="$(find turtlebot3_description)/urdf/turtlebot3_waffle.gazebo.xacro"/>
+  <xacro:include filename="$(find turtlebot3_description)/urdf/turtlebot3_gazebo.xacro"/>
   <xacro:property name="r200_cam_rgb_px" value="0.005"/>
   <xacro:property name="r200_cam_rgb_py" value="0.018"/>

File: urdf/turtlebot3_waffle_pi.urdf.xacro (robot description, xacro)
@@ -1,7 +1,9 @@
 <?xml version="1.0" ?>
 <robot name="turtlebot3_waffle_pi" xmlns:xacro="http://ros.org/wiki/xacro">
-  <xacro:arg name="prefix" default=""/>
-  <xacro:include filename="$(find turtlebot3_description)/urdf/common_properties.xacro"/>
-  <xacro:include filename="$(find turtlebot3_description)/urdf/turtlebot3_waffle_pi.gazebo.xacro"/>
+ <!-- Properties of waffle_pi -->
+ <xacro:property name="wheel_separation" value="0.287" />
+ <xacro:arg name="use_cam"    default="true"/>
+ <xacro:include filename="$(find turtlebot3_description)/urdf/common_properties.urdf"/>
+ <xacro:include filename="$(find turtlebot3_description)/urdf/turtlebot3_gazebo.xacro"/>
   <link name="$(arg prefix)base_footprint"/>
   <joint name="base_joint" type="fixed">
