Commit message: Initial support for Turtlebot3 in Ignition

File: urdf/turtlebot3_gazebo.xacro (robot description, xacro)
@@ -1,5 +1,5 @@
 <?xml version="1.0"?>
 <robot name="turtlebot3_gazebo" xmlns:xacro="http://ros.org/wiki/xacro">
-<!-- Argumens common to all turtlebots -->
+<!-- Arguments common to all turtlebots -->
  <xacro:arg name="laser_visual"  default="false"/>
  <xacro:arg name="camera_visual" default="false"/>
@@ -54,5 +54,5 @@
         <always_on>true</always_on>
         <visualize>$(arg imu_visual)</visualize>
-        <update_rate>200</update_rate>
+        <update_rate>50</update_rate>
         <imu>
           <angular_velocity>
@@ -106,5 +106,6 @@
   </gazebo>
  <gazebo>
-       <plugin name="turtlebot3_diff_drive" filename="libgazebo_ros_diff_drive.so">
+    <!-- classic -->
+    <plugin name="turtlebot3_diff_drive" filename="libgazebo_ros_diff_drive.so">
       <ros>
         <remapping>odom:=$(arg odom_topic)</remapping>
@@ -123,4 +124,14 @@
       <odometry_frame>$(arg prefix)odom</odometry_frame>
       <robot_base_frame>$(arg prefix)base_footprint</robot_base_frame>
+    </plugin>
+    <!-- Ignition -->
+    <plugin
+      filename="libignition-gazebo-diff-drive-system.so"
+      name="ignition::gazebo::systems::DiffDrive">
+      <left_joint>wheel_left_joint</left_joint>
+      <right_joint>wheel_right_joint</right_joint>
+      <wheel_separation>${wheel_separation}</wheel_separation>
+      <wheel_radius>0.033</wheel_radius>
+      <child_frame_id>$(arg prefix)base_footprint</child_frame_id>
     </plugin>
 </gazebo>
@@ -195,4 +206,5 @@
 </xacro:if>
    <gazebo>
+        <!-- classic -->
       <plugin name="turtlebot3_joint_state" filename="libgazebo_ros_joint_state_publisher.so">
       <ros>
@@ -204,4 +216,5 @@
       <joint_name>wheel_right_joint</joint_name>
     </plugin>
- </gazebo>
+      <plugin filename="libignition-gazebo-joint-state-publisher-system.so" name="ignition::gazebo::systems::JointStatePublisher"/>
+    </gazebo>
 </robot>

File: urdf/turtlebot3_waffle_pi.urdf.xacro (robot description, xacro)
@@ -16,5 +16,5 @@
       <origin xyz="-0.064 0 0.0" rpy="0 0 0"/>
       <geometry>
-        <mesh filename="package://turtlebot3_description/meshes/bases/waffle_pi_base.stl" scale="0.001 0.001 0.001"/>
+        <mesh filename="file://$(find turtlebot3_description)/meshes/bases/waffle_pi_base.stl" scale="0.001 0.001 0.001"/>
       </geometry>
       <material name="light_black"/>
@@ -44,5 +44,5 @@
       <origin xyz="0 0 0" rpy="1.57 0 0"/>
       <geometry>
-        <mesh filename="package://turtlebot3_description/meshes/wheels/left_tire.stl" scale="0.001 0.001 0.001"/>
+        <mesh filename="file://$(find turtlebot3_description)/meshes/wheels/left_tire.stl" scale="0.001 0.001 0.001"/>
       </geometry>
       <material name="dark"/>
@@ -72,5 +72,5 @@
       <origin xyz="0 0 0" rpy="1.57 0 0"/>
       <geometry>
-        <mesh filename="package://turtlebot3_description/meshes/wheels/right_tire.stl" scale="0.001 0.001 0.001"/>
+        <mesh filename="file://$(find turtlebot3_description)/meshes/wheels/right_tire.stl" scale="0.001 0.001 0.001"/>
       </geometry>
       <material name="dark"/>
@@ -145,5 +145,5 @@
       <origin xyz="0 0 0.0" rpy="0 0 0"/>
       <geometry>
-        <mesh filename="package://turtlebot3_description/meshes/sensors/lds.stl" scale="0.001 0.001 0.001"/>
+        <mesh filename="file://$(find turtlebot3_description)/meshes/sensors/lds.stl" scale="0.001 0.001 0.001"/>
       </geometry>
       <material name="dark"/>
